File: Kicad_data/SumNight57/right_key_matrix.kicad_sch (KiCad schematic)
At the start: 56 parts, among them SW1 SW_PUSH, SW10 SW_PUSH, SW11 SW_PUSH, SW12 SW_PUSH, SW13 SW_PUSH, SW14 SW_PUSH, SW15 SW_PUSH, SW16 SW_PUSH, SW17 SW_PUSH, SW18 SW_PUSH, SW19 SW_PUSH, SW2 SW_PUSH, SW20 SW_PUSH, SW21 SW_PUSH, SW22 SW_PUSH, SW23 SW_PUSH, SW24 SW_PUSH, SW25 SW_PUSH, SW26 SW_PUSH, SW27 SW_PUSH, SW28 SW_PUSH, SW3 SW_PUSH, SW4 SW_PUSH, SW5 SW_PUSH, SW6 SW_PUSH, SW7 SW_PUSH, SW8 SW_PUSH, SW9 SW_PUSH

Commit message: update
Connections:
- net Right_Col0: no longer SW25.1
- net Right_Col1: now also SW25.1; no longer SW26.1
- net Right_Col2: now also SW26.1; no longer SW27.1
- net Right_Col3: now also SW27.1; no longer SW28.1
- net Right_Col4: now also SW28.1
Other:
- moved on the sheet: D25, D26, D27, D28, SW25, SW26, SW27, SW28
